Commit message: fix params

File: p22_sensor_kit_description/urdf/sensor_kit.xacro (robot description, xacro)
@@ -4,11 +4,11 @@
     <xacro:arg name="gpu" default="false"/>
     <xacro:arg name="config_dir" default="$(find p22_sensor_kit_description)/config"/>
-    <xacro:property name="sensor_kit_base_link" default="sensor_kit_base_link"/>
-    <joint name="${sensor_kit_base_link}_joint" type="fixed">
+    <xacro:property name="sensor_kit" default="sensor_kit"/>
+    <joint name="${sensor_kit}_joint" type="fixed">
       <origin rpy="${roll} ${pitch} ${yaw}" xyz="${x} ${y} ${z}"/>
       <parent link="${parent}"/>
-      <child link="${sensor_kit_base_link}"/>
+      <child link="${sensor_kit}"/>
     </joint>
-    <link name="${sensor_kit_base_link}">
+    <link name="${sensor_kit}">
       <origin rpy="0 0 0" xyz="0 0 0"/>
     </link>

File: p22_sensor_kit_description/urdf/sensors.xacro (robot description, xacro)
@@ -7,10 +7,10 @@
   <xacro:sensor_kit_macro
     parent="base_link"
-    x="${calibration['base_link']['sensor_kit_base_link']['x']}"
-    y="${calibration['base_link']['sensor_kit_base_link']['y']}"
-    z="${calibration['base_link']['sensor_kit_base_link']['z']}"
-    roll="${calibration['base_link']['sensor_kit_base_link']['roll']}"
-    pitch="${calibration['base_link']['sensor_kit_base_link']['pitch']}"
-    yaw="${calibration['base_link']['sensor_kit_base_link']['yaw']}"
+    x="${calibration['base_link']['sensor_kit']['x']}"
+    y="${calibration['base_link']['sensor_kit']['y']}"
+    z="${calibration['base_link']['sensor_kit']['z']}"
+    roll="${calibration['base_link']['sensor_kit']['roll']}"
+    pitch="${calibration['base_link']['sensor_kit']['pitch']}"
+    yaw="${calibration['base_link']['sensor_kit']['yaw']}"
   />
 </robot>
